Commit message: chore: added dae models from openparallelgripper

File: genesis_lite6/assets/urdf/eef_ufgripper_ori.urdf (robot description, URDF)
Before this commit: robot eef_ufgripper, 4 links, 4 joints
Joints:
- joint finger_joint1: limit lower=0 upper=0.017 effort=5 velocity=2 -> lower=0 upper=0.0089 effort=5 velocity=2; origin xyz=0 0 0.07 rpy=0 0 0 -> xyz=0 0 0.0543 rpy=0 0 0
- joint finger_joint2: limit lower=0 upper=0.017 effort=5 velocity=2 -> lower=0 upper=0.0089 effort=5 velocity=2; origin xyz=0 0 0.07 rpy=0 0 0 -> xyz=0 0 0.0543 rpy=0 0 0
- joint joint_tcp: origin xyz=0 0 0.13 rpy=0 0 0 -> xyz=0 0 0.0836 rpy=0 0 0
